File: GPI-Tally-Interface-Board/GPI-Tally-Interface-Board.kicad_sch (KiCad schematic)
At the start: 43 parts, among them J1 DB25_Female, J2 DB25_Female, J8 THD-20-R, SW1 SW_Push_45deg, SW10 SW_Push_45deg, SW11 SW_Push_45deg, SW12 SW_Push_45deg, SW13 SW_Push_45deg, SW14 SW_Push_45deg, SW15 SW_Push_45deg, SW16 SW_Push_45deg, SW2 SW_Push_45deg, SW3 SW_Push_45deg, SW4 SW_Push_45deg, SW5 SW_Push_45deg, SW6 SW_Push_45deg, SW7 SW_Push_45deg, SW8 SW_Push_45deg, SW9 SW_Push_45deg, U1 BOB-12009, U2 BOB-12009, U3 BOB-12009, U4 BOB-12009

Commit message: oppto added
Parts:
- removed U1, U2, U3, U4: BOB-12009, CONV_BOB-12009, symbol BOB-12009:BOB-12009
- added J20: AMP171826-4, 171826-4:TE_171826-4, symbol Connector_Generic:Conn_01x04
- added R1, R10, R11, R12, R13, R14, R15, R16, R17, R18, R19, R2, R20, R21, R22, R23, R24, R25, R26, R27, R28, R29, R3, R30, R31, R32, R4, R5, R6, R7, R8, R9: 470, Resistor_SMD:R_0805_2012Metric_Pad1.20x1.40mm_HandSolder, symbol Device:R_Small
- added U10, U11, U12, U13, U14, U15, U16, U17, U18, U19, U20, U5, U6, U7, U8, U9: EL817, Package_DIP:DIP-4_W7.62mm, symbol Isolator:EL817
Connections:
- net +3.3V: now also SW1.1, R10.2, R11.2, R12.2, R13.2, R14.2, R15.2, R16.2, R25.2, R26.2, R27.2, R28.2, R29.2, R30.2, R31.2, R32.2, R9.2
- net A_GPI_OUT_1: now also R1.1
- net A_GPI_OUT_2: now also R2.1
- net A_GPI_OUT_3: now also R3.1
- net A_GPI_OUT_4: now also R4.1
- net A_GPI_OUT_5: now also R5.1
- net A_GPI_OUT_6: now also R6.1
- net A_GPI_OUT_7: now also R7.1
- net A_GPI_OUT_8: now also R8.1
- net B_GPI_OUT_1: now also R17.1
- net B_GPI_OUT_2: now also R18.1
- net B_GPI_OUT_3: now also R19.1
- net B_GPI_OUT_4: now also R20.1
- net B_GPI_OUT_5: now also R21.1
- net B_GPI_OUT_6: now also R22.1
- net B_GPI_OUT_7: now also R23.1
- net B_GPI_OUT_8: now also R24.1
- net GND: now also J20.2 (Pin_2), J20.3 (Pin_3), U10.3, U11.3, U12.3, U13.3, U14.3, U15.3, U16.3, U17.3, U18.3, U19.3, U20.3, U5.3, U6.3, U7.3, U8.3, U9.3; no longer J1.1, J1.11, J1.12, J1.13, J1.14 (P14), J1.15 (P15), J1.2, J1.24 (P24), J1.25 (P25), J2.1, J2.11, J2.12, J2.13, J2.14 (P14), J2.15 (P15), J2.2, J2.24 (P24), J2.25 (P25)
- net GPIO2: now also D1.1 (K), R9.1, U5.4
- net GPIO3: now also R10.1, U6.4
- net GPIO4: now also R11.1, U7.4
- net at D1.2 (A): now also SW1.2
- new net: R28.1, U16.4
- new net: R5.2, U9.1
- new net: R13.1, U9.4
- new net: R16.1, U12.4
- new net: R7.2, U11.1
- new net: R15.1, U11.4
- new net: R20.2, U16.1
- new net: R32.1, U20.4
- new net: R31.1, U19.4
- new net: R2.2, U6.1
- new net: R18.2, U14.1
- new net: R8.2, U12.1
- new net: R25.1, U13.4
- new net: R3.2, U7.1
- new net: R23.2, U19.1
- new net: R1.2, U5.1
- new net: R12.1, U8.4
- new net: R6.2, U10.1
- new net: R19.2, U15.1
- new net: R27.1, U15.4
- new net: R29.1, U17.4
- new net: R26.1, U14.4
- new net: R17.2, U13.1
- new net: R24.2, U20.1
- new net: R21.2, U17.1
- new net: R22.2, U18.1
- new net: R30.1, U18.4
- new net: R14.1, U10.4
- new net: R4.2, U8.1
- new net +12v: J20.1 (Pin_1)
- new net +5v: J20.4 (Pin_4)
- new net GND1: J1.1, J1.11, J1.12, J1.13, J1.14 (P14), J1.15 (P15), J1.2, J1.24 (P24), J1.25 (P25), U10.2, U11.2, U12.2, U5.2, U6.2, U7.2, U8.2, U9.2
- new net GND2: J2.1, J2.11, J2.12, J2.13, J2.14 (P14), J2.15 (P15), J2.2, J2.24 (P24), J2.25 (P25), U13.2, U14.2, U15.2, U16.2, U17.2, U18.2, U19.2, U20.2
Other:
- moved on the sheet: D1, D10, D11, D12, D13, D14, D15, D16, D2, D3, D4, D5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

Commit message: mirror
Parts:
- added D17: LED, LED_THT:LED_D5.0mm_IRGrey, symbol Device:LED
- added D18: LED, LED_THT:LED_D5.0mm_Clear, symbol Device:LED
- added R33, R34, R35, R36, R37, R38, R39, R40, R41, R42, R43, R44, R45, R46, R47, R48, R49, R50: 330, Resistor_SMD:R_0805_2012Metric_Pad1.20x1.40mm_HandSolder, symbol Device:R_Small
Connections:
- net +3.3V: now also R33.2, R34.2, R35.2, R36.2, R37.2, R38.2, R39.2, R40.2, R41.2, R42.2, R43.2, R44.2, R45.2, R46.2, R47.2, R48.2, R50.2; no longer SW1.1
- net GND: now also SW1.2, SW10.2, SW11.2, SW12.2, SW13.2, SW14.2, SW15.2, SW16.2, SW2.2, SW3.2, SW4.2, SW5.2, SW6.2, SW7.2, SW8.2, SW9.2, D17.1 (K), D18.1 (K)
- net GPIO10: now also D16.1 (K), R28.1, SW12.1, U16.4
- net GPIO11: now also D13.1 (K), R31.1, SW15.1, U19.4
- net GPIO14: now also D4.1 (K), R12.1, SW4.1, U8.4
- net GPIO15: now also D5.1 (K), R13.1, SW5.1, U9.4
- net GPIO17: now also D7.1 (K), R15.1, SW7.1, U11.4
- net GPIO18: now also D6.1 (K), R14.1, SW6.1, U10.4
- net GPIO2: now also SW1.1
- net GPIO20: now also R49.2
- net GPIO22: now also D9.1 (K), R25.1, SW9.1, U13.4
- net GPIO23: now also D10.1 (K), R26.1, SW10.1, U14.4
- net GPIO24: now also D11.1 (K), R27.1, SW11.1, U15.4
- net GPIO25: now also D14.1 (K), R30.1, SW14.1, U18.4
- net GPIO27: now also D8.1 (K), R16.1, SW8.1, U12.4
- net GPIO3: now also D2.1 (K), SW2.1
- net GPIO4: now also D3.1 (K), SW3.1
- net GPIO8: now also D12.1 (K), R32.1, SW16.1, U20.4
- net GPIO9: now also D15.1 (K), R29.1, SW13.1, U17.4
- net at D15.2 (A): now also R45.1
- net at D4.2 (A): now also R36.1
- net at D10.2 (A): now also R42.1
- net at D1.2 (A): now also R33.1; no longer SW1.2
- net at D3.2 (A): now also R35.1
- net at D11.2 (A): now also R43.1
- net at D8.2 (A): now also R40.1
- net at D16.2 (A): now also R44.1
- net at D12.2 (A): now also R48.1
- net at D13.2 (A): now also R47.1
- net at D14.2 (A): now also R46.1
- net at D9.2 (A): now also R41.1
- net at D7.2 (A): now also R39.1
- net at D6.2 (A): now also R38.1
- net at D5.2 (A): now also R37.1
- net at D2.2 (A): now also R34.1
- new net: D18.2 (A), R50.1
- new net: D17.2 (A), R49.1
Other:
- note added: "GPI Connector A"
- note added: "GPI Connector B"
- note added: "Rpi-GPIO"
- note added: "Test Buttons GPI A"
- note added: "Test Buttons GPI B"
- moved on the sheet: D1, D10, D11, D12, D13, D14, D15, D16, D2, D3, D4, D5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

Commit message: gerber
Connections:
- net GPIO10: now also D10.1 (K), R26.1, SW10.1, U14.4; no longer D16.1 (K), R28.1, SW12.1, U16.4
- net GPIO11: now also R29.1, SW13.1, U17.4; no longer R31.1, SW15.1, U19.4
- net GPIO17: now also D4.1 (K), R12.1, SW4.1, U8.4; no longer D7.1 (K), R15.1, SW7.1, U11.4
- net GPIO18: now also D5.1 (K), R13.1, SW5.1, U9.4; no longer D6.1 (K), R14.1, SW6.1, U10.4
- net GPIO22: now also D7.1 (K), R15.1, SW7.1, U11.4; no longer D9.1 (K), R25.1, SW9.1, U13.4
- net GPIO23: now also D8.1 (K), R16.1, SW8.1, U12.4; no longer D10.1 (K), R26.1, SW10.1, U14.4
- net GPIO24: now also D9.1 (K), R25.1, SW9.1, U13.4; no longer D11.1 (K), R27.1, SW11.1, U15.4
- net GPIO25: now also D12.1 (K), R28.1, SW12.1, U16.4; no longer D14.1 (K), R30.1, SW14.1, U18.4
- net GPIO27: now also D6.1 (K), R14.1, SW6.1, U10.4; no longer D8.1 (K), R16.1, SW8.1, U12.4
- net GPIO5: now also D16.1 (K), R32.1, SW16.1, U20.4
- net GPIO7: now also D15.1 (K), R31.1, SW15.1, U19.4
- net GPIO8: now also D14.1 (K), R30.1, SW14.1, U18.4; no longer D12.1 (K), R32.1, SW16.1, U20.4
- net GPIO9: now also D11.1 (K), R27.1, SW11.1, U15.4; no longer D15.1 (K), R29.1, SW13.1, U17.4
- removed net GPIO14: D4.1 (K), J8.8 (Pin_8), R12.1, SW4.1, U8.4
- removed net GPIO15: D5.1 (K), J8.10 (Pin_10), R13.1, SW5.1, U9.4
- new net RX: J8.10 (Pin_10)
- new net TX: J8.8 (Pin_8)
Other:
- moved on the sheet: D12, D13, D15, D16, R44, R45, R47, R48
